Commit message: up urdf

File: gazebo/eurobot2019/robots/eurobot2019.urdf (robot description, URDF)
Before this commit: robot eurobot2019, 1 links, 0 joints
Links:
- link base_link: geometry collision mesh filename=package://eurobot2019/meshes/base.dae; visual mesh filename=package://eurobot2019/meshes/base.dae

Commit message: up gazebo done

File: gazebo/eurobot2019/robots/eurobot2019.urdf (robot description, URDF)
Before this commit: robot eurobot2019, 1 links, 0 joints
Links:
- link base_link: geometry collision mesh filename=package://eurobot2019/meshes/base_link1.dae; visual mesh filename=package://eurobot2019/meshes/base_link1.dae

Commit message: up

File: gazebo/eurobot2019/robots/eurobot2019.urdf (robot description, URDF)
Before this commit: robot eurobot2019, 1 links, 0 joints
Links:
- added link world
Joints:
- added joint world_fixed: type fixed, parent world, child base_link
