Commit message: atom teat2

File: gazebo/eurobot2019/robots/eurobot2019_fixed.urdf (robot description, URDF)
Before this commit: robot eurobot2019, 2 links, 1 joints
Links:
- link base_link: mass 217.15 -> 1000
Joints:
- removed joint world_fixed
- added joint fixed: type fixed, parent world, child base_link
